File: Cad/bombhonor.brd (EAGLE design)
At the start: 64 x 61 mm, 0 parts

Commit message: Aggiunti tutti i pezzi tranne il connettore batteria ed il pulsante, domani fine schematico e calcolo costo per sapere se si fa o si muore
Parts:
- added 1, 2, U$1, U$2: (no value), AlmaPANEL:MOUSE_BITE_2MM
- added C1, C4: 10u, AlmaPASS:1206[3216]
- added C2, C3, C5, C6, C7, C8: 0.1u, AlmaPASS:0603[1608]
- added CN1: (no value), AlmaCONN:TC2030-IDC
- added LED1, LED10, LED11, LED12, LED13, LED14, LED15, LED16, LED17, LED18, LED19, LED2, LED20, LED21, LED22, LED23, LED24, LED25, LED26, LED27, LED28, LED29, LED3, LED30, LED4, LED5, LED6, LED7, LED8, LED9: RED, AlmaOPTO:1206[3216]BOTTOM_ENTRY
- added R1, R10, R11, R12, R13, R14, R15, R16, R17, R18, R19, R2, R20, R21, R22, R23, R24, R25, R26, R27, R28, R29, R3, R30, R31, R32, R4, R5, R6, R7, R8, R9: 1k, AlmaPASS:0603[1608]
- added U1: STM32F030F4, AlmaIC:TSSOP20
- added U3: LDO_EN, AlmaDCDC:SOT23-5
Connections:
- new net +3V3: C1.1, C2.1, C4.1, C5.1, C6.1, C7.1, C8.1, CN1.1, U1.16, U1.5, U3.5
- new net +5V: U3.1
- new net GND: C1.2, C2.2, C3.2, C4.2, C5.2, C6.2, C7.2, C8.2, CN1.5, LED1.K, LED10.K, LED11.K, LED12.K, LED13.K, LED14.K, LED15.K, LED16.K, LED17.K, LED18.K, LED19.K, LED2.K, LED20.K, LED21.K, LED22.K, LED23.K, LED24.K, LED25.K, LED26.K, LED27.K, LED28.K, LED29.K, LED3.K, LED30.K, LED4.K, LED5.K, LED6.K, LED7.K, LED8.K, LED9.K, R32.2, U1.1, U1.15, U3.2
- new net LED1: R1.2, R11.2, R16.2, R21.2, R26.2, R6.2, U1.8
- new net LED2: R12.2, R17.2, R2.2, R22.2, R27.2, R7.2, U1.9
- new net LED3: R13.2, R18.2, R23.2, R28.2, R3.2, R8.2, U1.10
- new net LED4: R14.2, R19.2, R24.2, R29.2, R4.2, R9.2, U1.11
- new net LED5: R10.2, R15.2, R20.2, R25.2, R30.2, R5.2, U1.12
- new net N$1: LED1.A, R1.1
- new net N$10: LED10.A, R10.1
- new net N$11: LED11.A, R11.1
- new net N$12: LED12.A, R12.1
- new net N$13: LED13.A, R13.1
- new net N$14: LED14.A, R14.1
- new net N$15: LED15.A, R15.1
- new net N$16: LED16.A, R16.1
- new net N$17: LED17.A, R17.1
- new net N$18: LED18.A, R18.1
- new net N$19: LED19.A, R19.1
- new net N$2: LED2.A, R2.1
- new net N$20: LED20.A, R20.1
- new net N$21: LED21.A, R21.1
- new net N$22: LED22.A, R22.1
- new net N$23: LED23.A, R23.1
- new net N$24: LED24.A, R24.1
- new net N$25: LED25.A, R25.1
- new net N$26: LED26.A, R26.1
- new net N$27: LED27.A, R27.1
- new net N$28: LED28.A, R28.1
- new net N$29: LED29.A, R29.1
- new net N$3: LED3.A, R3.1
- new net N$30: LED30.A, R30.1
- new net N$32: R31.1, R32.1, U3.3
- new net N$4: LED4.A, R4.1
- new net N$5: LED5.A, R5.1
- new net N$6: LED6.A, R6.1
- new net N$7: LED7.A, R7.1
- new net N$8: LED8.A, R8.1
- new net N$9: LED9.A, R9.1
- new net NRST: C3.1, CN1.3, U1.4
- new net ON: R31.2, U1.17
- new net SWCLK: CN1.4, U1.20
- new net SWDIO: CN1.2, U1.19
Other:
- board size 64 x 61 mm -> 66 x 62.8 mm

Commit message: Finito lo schematico. Mancano i parno per i passivi.
Parts:
- removed C7, C8: 0.1u, AlmaPASS:0603[1608]
- removed R32: 1k, AlmaPASS:0603[1608]
- removed U3: LDO_EN, AlmaDCDC:SOT23-5
- added BATT1: BK-883-TR, AlmaBATT:BK-883-TR
- added CN2: TR1-01, cesso:MAROGNATA
- CN1: value (none) -> HEADER4X1_2MM_SMD; device AlmaCONN:TC2030-IDC -> AlmaCONN:HEADER4X1_2MM_SMD
- moved R26 125.4 mm to (-18.0, -44.0)
- moved R27 125.4 mm to (-18.0, -48.0)
- moved R28 125.4 mm to (-18.0, -52.0)
- moved R29 125.4 mm to (-18.0, -56.0)
- moved R30 125.4 mm to (-18.0, -60.0)
- moved R31 120.1 mm to (-45.0, -88.0)
- moved R16 83.3 mm to (-30.0, -45.0)
- moved R17 83.3 mm to (-30.0, -49.0)
- moved R18 83.3 mm to (-30.0, -53.0)
- moved R19 83.3 mm to (-30.0, -57.0)
- moved R20 83.3 mm to (-30.0, -61.0)
- moved R21 83.3 mm to (-30.0, -65.0)
- moved R22 83.3 mm to (-30.0, -69.0)
- moved R23 83.3 mm to (-30.0, -73.0)
- moved R24 83.3 mm to (-30.0, -77.0)
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Connections:
- removed net +5V: U3.1
- removed net N$32: R31.1, R32.1, U3.3
- net +3V3: now also BATT1.V+1, CN1.4, CN2.1; no longer C7.1, C8.1, CN1.1, U3.5
- net GND: now also BATT1.V-, CN1.1, R31.1; no longer C7.2, C8.2, CN1.5, R32.2, U3.2
- net NRST: no longer CN1.3
- net ON: now also CN2.3
- net SWCLK: now also CN1.2; no longer CN1.4
- net SWDIO: now also CN1.3; no longer CN1.2

Commit message: Finito lo sbroglio della scheda
Parts:
- moved R25 113.7 mm to (27.2, 17.3), turned to 180 degrees
- moved R24 106.6 mm to (28.2, 12.3), turned to 180 degrees
- moved R4 105.6 mm to (-16.8, 23.6)
- moved R31 104.2 mm to (-16.0, 12.1)
- moved R3 101.3 mm to (-9.80, 21.6)
- moved CN2 101.0 mm to (-16.0, 17.0)
- moved R23 98.6 mm to (27.2, 7.30), turned to 180 degrees
- moved R1 96.4 mm to (0.10, 21.0)
- moved R2 95.8 mm to (-5.80, 18.6)
- moved C6 91.3 mm to (21.8, 5.80), turned to 270 degrees
- moved C5 91.0 mm to (17.0, 13.2), turned to 180 degrees
- moved R22 90.2 mm to (25.2, 2.30), turned to 180 degrees
- moved R30 86.3 mm to (4.20, 23.4)
- moved C4 86.1 mm to (17.0, 11.1), turned to 180 degrees
- moved R28 82.7 mm to (15.2, 23.7)
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Connections:
- net +3V3: now also BATT1.V+2; no longer BATT1.V+1
- net LED1: now also U1.6; no longer U1.8
- net LED2: now also U1.7; no longer U1.9
- net LED3: now also U1.8; no longer U1.10
- net LED4: now also U1.9; no longer U1.11
- net LED5: now also U1.10; no longer U1.12
- net ON: now also U1.2; no longer U1.17
Routing:
- net LED5: track 0.00 -> 206.5 mm, vias 0 -> 7
- net LED4: track 0.00 -> 202.4 mm, vias 0 -> 7
- net LED2: track 0.00 -> 198.4 mm, vias 0 -> 7
- net LED3: track 0.00 -> 195.9 mm, vias 0 -> 7
- net LED1: track 0.00 -> 186.1 mm, vias 0 -> 7
- net +3V3: track 0.00 -> 87.2 mm
- net ON: track 0.00 -> 32.5 mm, vias 0 -> 2
- net SWCLK: track 0.00 -> 25.6 mm
- net SWDIO: track 0.00 -> 20.2 mm
- net N$5: track 0.00 -> 3.17 mm
- net N$12: track 0.00 -> 3.14 mm
- net N$24: track 0.00 -> 3.11 mm
- net N$20: track 0.00 -> 3.11 mm
- net N$18: track 0.00 -> 3.10 mm
- net N$13: track 0.00 -> 3.10 mm
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- added copper zone on layer 1, net GND
- added copper zone on layer 16, net GND
